File: cape/6packRev1B.brd (EAGLE design)
At the start: 39.4 x 256.2 mm, 14 parts

Commit message: Make test cape more compact
Parts:
- moved ETHERNET1 50.8 mm to (19.1, 196.8)
- moved U$8 41.9 mm to (19.1, 172.7)
- moved U$7 35.6 mm to (19.1, 151.1)
- moved U$6 29.2 mm to (19.1, 129.5)
- moved U$5 22.9 mm to (19.1, 108.0)
- moved U$4 15.2 mm to (19.1, 86.4)
- moved U$3 8.89 mm to (19.1, 64.8)
- moved C4 6.35 mm to (20.3, 49.5)
- moved C3 5.08 mm to (20.3, 44.5)
- moved C1 3.81 mm to (16.5, 34.3)
- moved C2 3.81 mm to (16.5, 38.1)
Routing:
- net SDA2: track 243.3 -> 185.1 mm
- net GND2: track 233.2 -> 175.1 mm
- net SCL2: track 233.2 -> 176.4 mm
- net GND1: track 245.6 -> 193.7 mm
- net SCL1: track 244.9 -> 195.2 mm
- net +5V1: track 238.7 -> 191.7 mm
- net SDA1: track 238.8 -> 192.0 mm
- net +5V2: track 222.9 -> 189.4 mm
Other:
- board size 39.4 x 256.2 mm -> 34.3 x 206.7 mm

Commit message: Cape 1B try 2
Routing:
- net GND2: track 175.1 -> 222.1 mm, vias 0 -> 2
- net GND1: track 193.7 -> 230.1 mm
- net +5V1: track 191.7 -> 217.5 mm
- net +5V2: track 189.4 -> 172.3 mm
- net SDA2: track 185.1 -> 195.7 mm
- net SCL1: track 195.2 -> 200.9 mm
- net SDA1: track 192.0 -> 197.1 mm, vias 0 -> 2
- net SCL2: track 176.4 -> 177.2 mm
