File: cape/6packRev3A.brd (EAGLE design)
At the start: 38.1 x 209.2 mm, 16 parts

Commit message: Fix footprint cape 3A
Parts:
- R1, R2: device resistor:0207/10 -> resistor:0207/12
- moved R1 1.27 mm to (8.89, 24.1)
- moved R2 1.27 mm to (8.89, 29.2)
Routing:
- net +5V1: track 258.3 -> 261.0 mm
Changed lines of the file:
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@@
 <attribute name="VALUE" x="16.672" y="161.128" size="1.27" layer="27"/>
 </element>
-<element name="R1" library="resistor" library_urn="urn:adsk.eagle:library:348" package="0207/10" package3d_urn="urn:adsk.eagle:package:25939/1" value="4.7kΩ" x="10.16" y="24.13" rot="R180">
-<attribute name="NAME" x="13.208" y="22.606" size="1.27" layer="25" ratio="10" rot="R180"/>
-<attribute name="VALUE" x="12.4206" y="24.765" size="1.27" layer="27" ratio="10" rot="R180"/>
+<element name="R1" library="resistor" library_urn="urn:adsk.eagle:library:348" package="0207/12" package3d_urn="urn:adsk.eagle:package:25938/1" value="4.7kΩ" x="8.89" y="24.13" rot="R180">
+<attribute name="NAME" x="11.938" y="22.606" size="1.27" layer="25" ratio="10" rot="R180"/>
+<attribute name="VALUE" x="11.1506" y="24.765" size="1.27" layer="27" ratio="10" rot="R180"/>
 </element>
-<element name="R2" library="resistor" library_urn="urn:adsk.eagle:library:348" package="0207/10" package3d_urn="urn:adsk.eagle:package:25939/1" value="4.7kΩ" x="10.16" y="29.21" rot="R180">
-<attribute name="NAME" x="13.208" y="27.686" size="1.27" layer="25" ratio="10" rot="R180"/>
-<attribute name="VALUE" x="12.4206" y="29.845" size="1.27" layer="27" ratio="10" rot="R180"/>
+<element name="R2" library="resistor" library_urn="urn:adsk.eagle:library:348" package="0207/12" package3d_urn="urn:adsk.eagle:package:25938/1" value="4.7kΩ" x="8.89" y="29.21" rot="R180">
+<attribute name="NAME" x="11.938" y="27.686" size="1.27" layer="25" ratio="10" rot="R180"/>
+<attribute name="VALUE" x="11.1506" y="29.845" size="1.27" layer="27" ratio="10" rot="R180"/>
 </element>
 </elements>
@@
 <wire x1="16.6878" y1="15.09675625" x2="16.01824375" y2="14.4272" width="0.762" layer="16"/>
 <wire x1="16.01824375" y1="14.4272" x2="13.19175625" y2="14.4272" width="0.762" layer="16"/>
-<wire x1="13.19175625" y1="14.4272" x2="12.5222" y2="15.09675625" width="0.762" layer="16"/>
-<wire x1="12.5222" y1="15.09675625" x2="12.5222" y2="16.6878" width="0.762" layer="16"/>
-<wire x1="12.5222" y1="16.6878" x2="5.08" y2="24.13" width="0.762" layer="16"/>
 <wire x1="17.145" y1="16.51" x2="16.6878" y2="16.0528" width="0.762" layer="16"/>
 <wire x1="16.6878" y1="16.0528" x2="16.6878" y2="15.09675625" width="0.762" layer="16"/>
-<wire x1="5.08" y1="24.13" x2="5.08" y2="29.21" width="0.762" layer="16"/>
-<wire x1="8.255" y1="35.84108125" x2="9.37091875" y2="36.957" width="0.762" layer="16"/>
 <wire x1="13.48908125" y1="36.957" x2="14.605" y2="35.84108125" width="0.762" layer="16"/>
-<wire x1="5.08" y1="29.21" x2="8.255" y2="32.385" width="0.762" layer="16"/>
 <wire x1="14.605" y1="35.84108125" x2="14.605" y2="34.925" width="0.762" layer="16"/>
 <wire x1="14.605" y1="34.925" x2="15.24" y2="34.29" width="0.762" layer="16"/>
-<wire x1="8.255" y1="32.385" x2="8.255" y2="35.84108125" width="0.762" layer="16"/>
 <wire x1="9.37091875" y1="36.957" x2="13.48908125" y2="36.957" width="0.762" layer="16"/>
+<wire x1="13.19175625" y1="14.4272" x2="3.48895625" y2="24.13" width="0.762" layer="16"/>
+<wire x1="3.48895625" y1="24.13" x2="2.54" y2="24.13" width="0.762" layer="16"/>
+<wire x1="2.54" y1="24.13" x2="2.54" y2="29.21" width="0.762" layer="16"/>
+<wire x1="2.54" y1="29.21" x2="8.255" y2="34.925" width="0.762" layer="16"/>
+<wire x1="8.255" y1="34.925" x2="8.255" y2="35.84108125" width="0.762" layer="16"/>
+<wire x1="8.255" y1="35.84108125" x2="9.37091875" y2="36.957" width="0.762" layer="16"/>
 </signal>
 <signal name="GND1">
@@
 <wire x1="14.605" y1="16.51" x2="14.605" y2="17.374475" width="0.762" layer="16"/>
 <wire x1="14.605" y1="17.374475" x2="13.7922" y2="18.187275" width="0.762" layer="16"/>
+<wire x1="10.795" y1="33.655" x2="10.16" y2="34.29" width="0.762" layer="16"/>
 <wire x1="13.7922" y1="18.187275" x2="13.7922" y2="22.6822" width="0.762" layer="16"/>
 <wire x1="13.7922" y1="22.6822" x2="15.24" y2="24.13" width="0.762" layer="16"/>
-<wire x1="10.795" y1="33.655" x2="10.16" y2="34.29" width="0.762" layer="16"/>
-<wire x1="15.24" y1="24.13" x2="15.24" y2="26.65960625" width="0.762" layer="16"/>
-<wire x1="15.24" y1="26.65960625" x2="10.795" y2="31.10460625" width="0.762" layer="16"/>
-<wire x1="10.795" y1="31.10460625" x2="10.795" y2="33.655" width="0.762" layer="16"/>
+<wire x1="15.24" y1="24.13" x2="10.795" y2="28.575" width="0.762" layer="16"/>
+<wire x1="10.795" y1="28.575" x2="10.795" y2="33.655" width="0.762" layer="16"/>
 </signal>
 <signal name="SDA1">
@@
 <wire x1="17.0434" y1="23.38300625" x2="17.0434" y2="27.4066" width="0.762" layer="16"/>
 <wire x1="17.0434" y1="27.4066" x2="15.24" y2="29.21" width="0.762" layer="16"/>
-<wire x1="15.24" y1="29.21" x2="12.7" y2="31.75" width="0.762" layer="16"/>
-<wire x1="12.7" y1="31.75" x2="12.7" y2="34.29" width="0.762" layer="16"/>
+<wire x1="13.335" y1="32.73891875" x2="13.335" y2="33.655" width="0.762" layer="16"/>
+<wire x1="13.335" y1="33.655" x2="12.7" y2="34.29" width="0.762" layer="16"/>
+<wire x1="15.24" y1="29.21" x2="15.24" y2="30.83391875" width="0.762" layer="16"/>
+<wire x1="15.24" y1="30.83391875" x2="13.335" y2="32.73891875" width="0.762" layer="16"/>
 </signal>
 <signal name="GND2">
